File: PCB/LimeShield-kicad/file5471FB9C.sch (KiCad schematic (older format))
At the start: 10 parts

Commit message: added GPIO-2 on PCB, most things are unrouted, finished conversion from eagle
Parts:
- C41: renamed from C42; footprint Capacitors_SMD:C_0402 -> Capacitors_SMD:C_0805
- C42: renamed from C41; footprint Capacitors_SMD:C_0402 -> Capacitors_SMD:C_0805
Changed lines of the file:
@@
 Sheet 3 3
 Title "Videobrick"
-Date "2015-02-05"
-Rev "alpha 4"
-Comp ""
+Date "2015-02-06"
+Rev "alpha 5"
+Comp "OTELOeGen"
 Comment1 "by Mechatronik Karl Zeilhofer"
 Comment2 "Transfered from Eagle to KiCad"
@@
 AR Path="/5471FB42/5471FB9D/54722431" Ref="C?"  Part="1"
 AR Path="/54724AE0/54722431" Ref="C?"  Part="1"
-AR Path="/54725066/54722431" Ref="C42"  Part="1"
-F 0 "C42" H 2750 6000 40  0000 L CNN
+AR Path="/54725066/54722431" Ref="C41"  Part="1"
+F 0 "C41" H 2750 6000 40  0000 L CNN
 F 1 "10u" H 2756 5815 40  0000 L CNN
-F 2 "Capacitors_SMD:C_0402" H 2788 5750 30  0001 C CNN
+F 2 "Capacitors_SMD:C_0805" H 2788 5750 30  0001 C CNN
 F 3 "" H 2750 5900 60  0000 C CNN
 	1    2750 5900
@@
 P 3050 6100
 AR Path="/54724AE0/547224CB" Ref="C?"  Part="1"
-AR Path="/54725066/547224CB" Ref="C41"  Part="1"
-F 0 "C41" H 3050 6200 40  0000 L CNN
+AR Path="/54725066/547224CB" Ref="C42"  Part="1"
+F 0 "C42" H 3050 6200 40  0000 L CNN
 F 1 "10u" H 3056 6015 40  0000 L CNN
-F 2 "Capacitors_SMD:C_0402" H 3088 5950 30  0001 C CNN
+F 2 "Capacitors_SMD:C_0805" H 3088 5950 30  0001 C CNN
 F 3 "" H 3050 6100 60  0000 C CNN
 	1    3050 6100
@@
 	11800 5750 13800 5750
 Wire Wire Line
-	11100 4550 9700 4550
+	9700 4550 11100 4550
 Wire Wire Line
 	9700 4550 9700 4250
